Commit message: Add camera collision object and params, mimic joints

File: urdf/exoter.urdf (robot description, URDF)
Before this commit: robot exoter, 32 links, 31 joints
Links:
- link camera_assembly: geometry collision box size=0.075013 0.157175 0.1385; visual mesh filename=../meshes/Bb2 And Tof Camera.obj scale=1.0 1.0 1.0
